File: arduino_Uno_Rev3-02-TH.brd (EAGLE design)
At the start: 73.7 x 33 mm, 28 parts, among them IC1 7805T, Q1 16MHz, X1 POWERSUPPLY_DC21MMX, X2 Ser_Comm, X3 POWER

Commit message: Second revision of the breadboard-mountable Arduino
Second revision of the breadboard-mountable Arduino, making use of
better parts (using Adafruit and Sparkfun libraries) and positioning
silkscreen smartly.
Parts:
- removed AD: 6x1F-H8.5, SmartPrj:1X06
- removed IOH: 22-23-2081, con-molex:22-23-2081
- removed IOL: 8x1F-H8.5, SmartPrj:1X08
- removed X2: Ser_Comm, con-molex:22-23-2061
- removed X3: POWER, con-molex:22-23-2061
- added JP1, JP3, JP5: (no value), adafruit:1X06
- added JP2, JP4: (no value), adafruit:1X08-BIG
Connections:
- net +5V: now also JP3.3, JP5.4; no longer X2.4, X3.3
- net AD0: now also JP1.6; no longer AD.1
- net AD1: now also JP1.5; no longer AD.2
- net AD2: now also JP1.4; no longer AD.3
- net AD3: now also JP1.3; no longer AD.4
- net AD4/SDA: now also JP1.2; no longer AD.5
- net AD5/SCL: now also JP1.1; no longer AD.6
- net AREF: now also JP4.1; no longer IOH.1
- net DTR: now also JP5.1; no longer X2.1
- net GND: now also JP3.4, JP3.5, JP4.2, JP5.6; no longer IOH.2, X2.6, X3.4, X3.5
- net IO0: now also JP2.8; no longer IOL.1
- net IO1: now also JP2.7; no longer IOL.2
- net IO2: now also JP2.6; no longer IOL.3
- net IO3: now also JP2.5; no longer IOL.4
- net IO4: now also JP2.4; no longer IOL.5
- net IO5: now also JP2.3; no longer IOL.6
- net IO6: now also JP2.2; no longer IOL.7
- net IO7: now also JP2.1; no longer IOL.8
- net IO8: now also JP4.8; no longer IOH.8
- net IO9: now also JP4.7; no longer IOH.7
- net M8RXD: now also JP5.3; no longer X2.3
- net M8TXD: now also JP5.2; no longer X2.2
- net MISO: now also JP4.4; no longer IOH.4
- net MOSI: now also JP4.5; no longer IOH.5
- net N$1: now also JP3.2; no longer X3.2
- net N$8: now also JP5.5; no longer X2.5
- net RESET: now also JP3.1; no longer X3.1
- net SCK: now also JP4.3; no longer IOH.3
- net SS: now also JP4.6; no longer IOH.6
- net VIN: now also JP3.6; no longer X3.6
Routing:
- net GND: track 93.0 -> 76.5 mm, vias 21 -> 20
- net VIN: track 35.8 -> 39.0 mm
- net MISO: track 51.8 -> 51.2 mm
Other:
- board text added: "Fritzen Proto"
- board text removed: "#"
- board text removed: "3V3"
- board text removed: "ANALOG IN"
- board text removed: "ATMEGA328"
- board text removed: "Arduino"
- board text removed: "C9"
- board text removed: "D.Cuartielles"
- board text removed: "D.Mellis"
- board text removed: "DIGITAL"
- board text removed: "Fritzen UM"
- board text removed: "G.Martino"
- board text removed: "IOREF"
- board text removed: "ITALY"
- board text removed: "L"
- board text removed: "LED1"
- board text removed: "M.Banzi"
- board text removed: "MADE IN"
- board text removed: "MCU"
- board text removed: "ON"
- board text removed: "PC1"
- board text removed: "PC2"
- board text removed: "RESET"
- board text removed: "RX"
- board text removed: "Rst"
- board text removed: "S1"
- board text removed: "SCL"
- board text removed: "SDA"
- board text removed: "T.Igoe"
- board text removed: "TM"
- board text removed: "TX"
- board text removed: "UNO"
- board text removed: "VIN"
- board text removed: "[#=PWM]"
- board text removed: "designed by"
- board text removed: "tinker it"
- board text removed: "www.arduino.cc"
