File: arduino_Uno_Rev3-02-TH.sch (EAGLE design)
At the start: 28 parts, among them IC1 7805T, Q1 16MHz, X1 POWERSUPPLY_DC21MMX, X2 Ser_Comm, X3 POWER

Commit message: Second revision of the breadboard-mountable Arduino
Second revision of the breadboard-mountable Arduino, making use of
better parts (using Adafruit and Sparkfun libraries) and positioning
silkscreen smartly.
Parts:
- removed AD: 6x1F-H8.5, SmartPrj:PINHD-1X6
- removed IOH: 22-23-2081, con-molex:22-23-2081
- removed IOL: 8x1F-H8.5, SmartPrj:PINHD-1X8
- removed X2: Ser_Comm, con-molex:22-23-2061
- removed X3: POWER, con-molex:22-23-2061
- added JP1, JP3, JP5: (no value), adafruit:PINHD-1X6
- added JP2, JP4: (no value), adafruit:PINHD-1X8BIG
Connections:
- net +5V: now also JP3.3, JP5.4; no longer X2-4.S, X3-3.S
- net AD0: now also JP1.6; no longer AD.1
- net AD1: now also JP1.5; no longer AD.2
- net AD2: now also JP1.4; no longer AD.3
- net AD3: now also JP1.3; no longer AD.4
- net AD4/SDA: now also JP1.2; no longer AD.5
- net AD5/SCL: now also JP1.1; no longer AD.6
- net AREF: now also JP4.1; no longer IOH-1.S
- net DTR: now also JP5.1; no longer X2-1.S
- net GND: now also JP3.4, JP3.5, JP4.2, JP5.6; no longer IOH-2.S, X2-6.S, X3-4.S, X3-5.S
- net IO0: now also JP2.8; no longer IOL.1
- net IO1: now also JP2.7; no longer IOL.2
- net IO2: now also JP2.6; no longer IOL.3
- net IO3: now also JP2.5; no longer IOL.4
- net IO4: now also JP2.4; no longer IOL.5
- net IO5: now also JP2.3; no longer IOL.6
- net IO6: now also JP2.2; no longer IOL.7
- net IO7: now also JP2.1; no longer IOL.8
- net IO8: now also JP4.8; no longer IOH-8.S
- net IO9: now also JP4.7; no longer IOH-7.S
- net M8RXD: now also JP5.3; no longer X2-3.S
- net M8TXD: now also JP5.2; no longer X2-2.S
- net MISO: now also JP4.4; no longer IOH-4.S
- net MOSI: now also JP4.5; no longer IOH-5.S
- net N$1: now also JP3.2; no longer X3-2.S
- net N$8: now also JP5.5; no longer X2-5.S
- net RESET: now also JP3.1; no longer X3-1.S
- net SCK: now also JP4.3; no longer IOH-3.S
- net SS: now also JP4.6; no longer IOH-6.S
- net VIN: now also JP3.6; no longer X3-6.S
Other:
- note removed: "Arduino(TM) UNO Rev3"

Commit message: Third revision and Fabrication Files
I have ordered 30 pieces of this PCB at MakerStudio.CC on 03/23/2016
Parts:
- JP1: value (none) -> AD
- JP2: value (none) -> IOL
- JP3: value (none) -> POWER
- JP4: value (none) -> IOH
- JP5: value (none) -> COMM
Connections:
- removed net N$8: JP5.5
- net RESET: now also JP5.5
Changed lines of the file:
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@@
 <layer number="59" name="tCarbon" color="7" fill="1" visible="no" active="no"/>
 <layer number="60" name="bCarbon" color="7" fill="1" visible="no" active="no"/>
-<layer number="90" name="Modules" color="7" fill="1" visible="no" active="yes"/>
+<layer number="90" name="Modules" color="7" fill="1" visible="yes" active="yes"/>
 <layer number="91" name="Nets" color="2" fill="1" visible="yes" active="yes"/>
 <layer number="92" name="Busses" color="1" fill="1" visible="yes" active="yes"/>
@@
 <layer number="106" name="bPlate" color="7" fill="1" visible="yes" active="yes"/>
 <layer number="107" name="Crop" color="7" fill="1" visible="yes" active="yes"/>
-<layer number="108" name="fp8" color="7" fill="1" visible="no" active="yes"/>
-<layer number="109" name="fp9" color="7" fill="1" visible="no" active="yes"/>
-<layer number="110" name="fp0" color="7" fill="1" visible="no" active="yes"/>
-<layer number="111" name="LPC17xx" color="7" fill="1" visible="no" active="yes"/>
-<layer number="112" name="tSilk" color="7" fill="1" visible="no" active="yes"/>
+<layer number="108" name="fp8" color="7" fill="1" visible="yes" active="yes"/>
+<layer number="109" name="fp9" color="7" fill="1" visible="yes" active="yes"/>
+<layer number="110" name="fp0" color="7" fill="1" visible="yes" active="yes"/>
+<layer number="111" name="LPC17xx" color="7" fill="1" visible="yes" active="yes"/>
+<layer number="112" name="tSilk" color="7" fill="1" visible="yes" active="yes"/>
 <layer number="113" name="ReferenceLS" color="7" fill="1" visible="no" active="no"/>
 <layer number="116" name="Patch_BOT" color="7" fill="1" visible="yes" active="yes"/>
@@
 <layer number="121" name="_tsilk" color="7" fill="1" visible="yes" active="yes"/>
 <layer number="122" name="_bsilk" color="7" fill="1" visible="yes" active="yes"/>
-<layer number="123" name="tTestmark" color="7" fill="1" visible="no" active="yes"/>
-<layer number="124" name="bTestmark" color="7" fill="1" visible="no" active="yes"/>
-<layer number="125" name="_tNames" color="7" fill="1" visible="no" active="yes"/>
-<layer number="126" name="_bNames" color="7" fill="1" visible="no" active="yes"/>
-<layer number="127" name="_tValues" color="7" fill="1" visible="no" active="yes"/>
-<layer number="128" name="_bValues" color="7" fill="1" visible="no" active="yes"/>
+<layer number="123" name="tTestmark" color="7" fill="1" visible="yes" active="yes"/>
+<layer number="124" name="bTestmark" color="7" fill="1" visible="yes" active="yes"/>
+<layer number="125" name="_tNames" color="7" fill="1" visible="yes" active="yes"/>
+<layer number="126" name="_bNames" color="7" fill="1" visible="yes" active="yes"/>
+<layer number="127" name="_tValues" color="7" fill="1" visible="yes" active="yes"/>
+<layer number="128" name="_bValues" color="7" fill="1" visible="yes" active="yes"/>
 <layer number="129" name="Mask" color="7" fill="1" visible="yes" active="yes"/>
-<layer number="131" name="tAdjust" color="7" fill="1" visible="no" active="yes"/>
-<layer number="132" name="bAdjust" color="7" fill="1" visible="no" active="yes"/>
+<layer number="131" name="tAdjust" color="7" fill="1" visible="yes" active="yes"/>
+<layer number="132" name="bAdjust" color="7" fill="1" visible="yes" active="yes"/>
 <layer number="144" name="Drill_legend" color="7" fill="1" visible="yes" active="yes"/>
-<layer number="150" name="Notes" color="7" fill="1" visible="no" active="yes"/>
+<layer number="150" name="Notes" color="7" fill="1" visible="yes" active="yes"/>
 <layer number="151" name="HeatSink" color="7" fill="1" visible="yes" active="yes"/>
-<layer number="152" name="_bDocu" color="7" fill="1" visible="no" active="yes"/>
+<layer number="152" name="_bDocu" color="7" fill="1" visible="yes" active="yes"/>
 <layer number="153" name="FabDoc1" color="6" fill="1" visible="no" active="no"/>
 <layer number="154" name="FabDoc2" color="2" fill="1" visible="no" active="no"/>
 <layer number="155" name="FabDoc3" color="7" fill="15" visible="no" active="no"/>
-<layer number="199" name="Contour" color="7" fill="1" visible="no" active="yes"/>
+<layer number="199" name="Contour" color="7" fill="1" visible="yes" active="yes"/>
 <layer number="200" name="200bmp" color="1" fill="10" visible="no" active="no"/>
 <layer number="201" name="201bmp" color="7" fill="1" visible="yes" active="yes"/>
@@
 <layer number="232" name="Eagle3D_PG2" color="7" fill="1" visible="no" active="no"/>
 <layer number="233" name="Eagle3D_PG3" color="7" fill="1" visible="no" active="no"/>
-<layer number="248" name="Housing" color="7" fill="1" visible="no" active="yes"/>
-<layer number="249" name="Edge" color="7" fill="1" visible="no" active="yes"/>
+<layer number="248" name="Housing" color="7" fill="1" visible="yes" active="yes"/>
+<layer number="249" name="Edge" color="7" fill="1" visible="yes" active="yes"/>
 <layer number="250" name="Descript" color="3" fill="1" visible="no" active="no"/>
 <layer number="251" name="SMDround" color="12" fill="11" visible="no" active="no"/>
@@
 <part name="R6" library="rcl" deviceset="R-EU_" device="0207/10" value="1k"/>
 <part name="C2" library="capacitor-wima" deviceset="C" device="2,5-3" value="100nF"/>
-<part name="JP1" library="adafruit" deviceset="PINHD-1X6" device=""/>
-<part name="JP2" library="adafruit" deviceset="PINHD-1X8" device="BIG"/>
-<part name="JP3" library="adafruit" deviceset="PINHD-1X6" device=""/>
-<part name="JP4" library="adafruit" deviceset="PINHD-1X8" device="BIG"/>
-<part name="JP5" library="adafruit" deviceset="PINHD-1X6" device=""/>
+<part name="JP1" library="adafruit" deviceset="PINHD-1X6" device="" value="AD"/>
+<part name="JP2" library="adafruit" deviceset="PINHD-1X8" device="BIG" value="IOL"/>
+<part name="JP3" library="adafruit" deviceset="PINHD-1X6" device="" value="POWER"/>
+<part name="JP4" library="adafruit" deviceset="PINHD-1X8" device="BIG" value="IOH"/>
+<part name="JP5" library="adafruit" deviceset="PINHD-1X6" device="" value="COMM"/>
 </parts>
 <sheets>
@@
 <pinref part="JP3" gate="A" pin="1"/>
 </segment>
+<segment>
+<wire x1="96.52" y1="154.94" x2="99.06" y2="154.94" width="0.1524" layer="91"/>
+<pinref part="JP5" gate="A" pin="5"/>
+<label x="101.6" y="154.94" size="1.778" layer="95"/>
+</segment>
 </net>
 <net name="VIN" class="1">
@@
 </segment>
 </net>
-<net name="N$8" class="0">
-<segment>
-<wire x1="96.52" y1="154.94" x2="99.06" y2="154.94" width="0.1524" layer="91"/>
-<pinref part="JP5" gate="A" pin="5"/>
-</segment>
-</net>
